Commit message: feat(description): 로봇 바퀴 모델링 및 xacro 매크로 구현
- Xacro Property를 이용한 기하학적 상수 정의
- 반복되는 바퀴 모델링을 위한 wheel 매크로 구현
- 4개 바퀴에 대한 continuous joint 설정 완료
- RViz2 material 파싱 에러 수정을 위해 name 속성 추가
- Step4 학습 내용 LEARNING.md 업데이트

File: src/gyubot_description/urdf/gyubot.urdf.xacro (robot description, xacro)
@@ -1,16 +1,55 @@
 <?xml version="1.0"?>
-<robot name="gyubot" xmlns:xacro="http://www.ros.rog/wiki/xacro">
-    <!-- Base Link 로봇의 물리적/기하학적 중심이 되는 최초의 뼈대입니다. -->
-     <link name="base_link">
+<robot name="gyubot" xmlns:xacro="http://www.ros.org/wiki/xacro">
+    <!-- 1. 상수 정의 (Properties) -->
+    <!-- 치수를 변수로 관리하면 나중에 로봇 크기를 바꿀 때 매우 편리함-->
+    <xacro:property name="base_width" value="0.4" />
+    <xacro:property name="base_length" value="0.5" />
+    <xacro:property name="base_height" value="0.2" />
+    <xacro:property name="wheel_radius" value="0.10" />
+    <xacro:property name="wheel_width" value="0.05" />
+    <xacro:property name="wheel_ygap" value="0.025" /> <!-- 본체와 바퀴 사이의 유격-->
+    <!-- 바퀴 중심 위치(Offset) 계산 -->
+    <xacro:property name="wheel_xoff" value="0.15" />
+    <xacro:property name="wheel_yoff" value="${base_width/2 + wheel_width/2 + wheel_ygap}"/>
+    <xacro:property name="wheel_zoff" value="0.05" />
+    <!-- 2. Base Link 정의 -->
+    <link name="base_link">
         <visual>
-            <!-- 크기가 x: 0.5m, y: 0.4m, z: 0.2m 인 직육면체 상자를 표현합니다. -->
             <geometry>
-                <box size="0.5 0.4 0.2"/>
+                <box size="${base_length} ${base_width} ${base_height}"/>
             </geometry>
-            <!-- 로봇 본체의 색상을 파란색으로 지정합니다. (R, G, B, Alpha) -->
             <material name="blue">
                 <color rgba="0.0 0.0 0.8 1.0"/>
             </material>
         </visual>
-     </link>
+    </link>
+    <!-- 3. 바퀴 매크로 (Wheel Macro) -->
+    <!-- 매크로는 프로그래밍의 '함수'와 같다. 바퀴 4개를 일일이 코딩하지 않고 이 틀을 사용함-->
+    <xacro:macro name="wheel" params="prefix x_reflect y_reflect">
+        <link name="${prefix}_wheel">
+            <visual>
+                <!-- Cylinder는 기본적으로 위아래로 서 있다. rpy="${pi/2} 0 0"으로 90도 눕혀준다.-->
+                 <origin xyz="0 0 0" rpy="${pi/2} 0 0"/>
+                 <geometry>
+                    <cylinder radius="${wheel_radius}" length="${wheel_width}"/>
+                 </geometry>
+                 <material name="black">
+                    <color rgba="0.0 0.0 0.0 1.0"/>
+                 </material>
+            </visual>
+        </link>
+        <!-- Joint: base_link와 바퀴를 연결 -->
+        <joint name="${prefix}_joint" type="continuous">
+            <parent link="base_link"/>
+            <child link="${prefix}_wheel"/>
+            <!-- x_reflect, y_reflect을 이용해 4군데 위치를 결정한다. -->
+            <origin xyz="${x_reflect*wheel_xoff} ${y_reflect*wheel_yoff} ${-wheel_zoff}" rpy="0 0 0" />
+            <axis xyz="0 1 0 "/> <!-- 바퀴가 회전하는 축 (y축) -->
+        </joint>
+    </xacro:macro>
+    <!-- 4. 매크로 호출 (4개의 바퀴 생성) -->
+    <xacro:wheel prefix="front_left" x_reflect="1" y_reflect="1" />
+    <xacro:wheel prefix="front_right" x_reflect="1" y_reflect="-1" />
+    <xacro:wheel prefix="rear_left" x_reflect="-1" y_reflect="1" />
+    <xacro:wheel prefix="rear_right" x_reflect="-1" y_reflect="-1" />
 </robot>

Commit message: refactor(description): 바퀴 인디케이터 링크 분리 및 재질 구조 최적화
- URDF 내 여러 visual 요소 병합 시 발생하는 색상 상속(간섭) 문제 해결을 위해 인디케이터를 독립된 링크로 분리
- 바퀴 링크와 인디케이터 링크를 fixed joint로 연결하여 회전 동기화
- Material 정의를 전역으로 분리하여 코드 재사용성 및 이름 충돌 방지
- docs: LEARNING.md Box size 의미 및 링크 분리 트러블슈팅 기록 추가(Step5)

File: src/gyubot_description/urdf/gyubot.urdf.xacro (robot description, xacro)
@@ -13,5 +13,15 @@
     <xacro:property name="wheel_yoff" value="${base_width/2 + wheel_width/2 + wheel_ygap}"/>
     <xacro:property name="wheel_zoff" value="0.05" />
-    <!-- 2. Base Link 정의 -->
+    <!-- 2. 재질(Material) 정의 -->
+    <material name="blue">
+        <color rgba="0.0 0.0 0.8 1.0"/>
+    </material>
+    <material name="black">
+        <color rgba="0.0 0.0 0.0 1.0"/>
+    </material>
+    <material name="white">
+        <color rgba="1.0 1.0 1.0 1.0"/>
+    </material>
+    <!-- 3. Base Link 정의 -->
     <link name="base_link">
         <visual>
@@ -19,10 +29,8 @@
                 <box size="${base_length} ${base_width} ${base_height}"/>
             </geometry>
-            <material name="blue">
-                <color rgba="0.0 0.0 0.8 1.0"/>
-            </material>
+            <material name="blue"/>
         </visual>
     </link>
-    <!-- 3. 바퀴 매크로 (Wheel Macro) -->
+    <!-- 4. 바퀴 매크로 (Wheel Macro) -->
     <!-- 매크로는 프로그래밍의 '함수'와 같다. 바퀴 4개를 일일이 코딩하지 않고 이 틀을 사용함-->
     <xacro:macro name="wheel" params="prefix x_reflect y_reflect">
@@ -34,9 +42,25 @@
                     <cylinder radius="${wheel_radius}" length="${wheel_width}"/>
                  </geometry>
-                 <material name="black">
-                    <color rgba="0.0 0.0 0.0 1.0"/>
-                 </material>
+                 <material name="black"/>
             </visual>
         </link>
+        <!-- 회전 확인용 인디케이터 (별도 링크로 분리) -->
+        <!-- Gazebo 등 일부 환경에서는 하나의 링크에 여러 visual이 있을 경우 재질이 하나로 통일되는 문제가 있음 -->
+        <!-- 이를 해결하기 위해 별도의 링크로 분리하고 fixed joint로 연결함 -->
+        <link name="${prefix}_wheel_indicator">
+            <visual>
+                <origin xyz="0 0 0" rpy="${pi/2} 0 0"/>
+                <geometry>
+                    <!-- 바퀴 옆면에 붙은 작은 사각형 -->
+                     <box size="0.03 0.01 ${wheel_width + 0.002}"/>
+                </geometry>
+                <material name="white"/>
+            </visual>
+        </link>
+        <joint name="${prefix}_indicator_joint" type="fixed">
+            <parent link="${prefix}_wheel"/>
+            <child link="${prefix}_wheel_indicator"/>
+            <origin xyz="${wheel_radius - 0.02} 0 0" rpy="0 0 0"/>
+        </joint>
         <!-- Joint: base_link와 바퀴를 연결 -->
         <joint name="${prefix}_joint" type="continuous">
@@ -48,5 +72,5 @@
         </joint>
     </xacro:macro>
-    <!-- 4. 매크로 호출 (4개의 바퀴 생성) -->
+    <!-- 5. 매크로 호출 (4개의 바퀴 생성) -->
     <xacro:wheel prefix="front_left" x_reflect="1" y_reflect="1" />
     <xacro:wheel prefix="front_right" x_reflect="1" y_reflect="-1" />

Commit message: feat(description): Gazebo 시뮬레이션 환경 구축 및 구동 플러그인 추가
- URDF에 box/cylinder 관성(Inertia) 계산 매크로 추가
- base_link 및 wheel 링크에 collision 속성 적용
- libgazebo_ros_diff_drive 플러그인으로 skid_steer 구동 구현
- CMakeLists.txt install() 블록 위치 최적화
- LEARNING.md Step 6 Gazebo 시뮬레이션 학습 내용 기록

File: src/gyubot_description/urdf/gyubot.urdf.xacro (robot description, xacro)
@@ -13,4 +13,19 @@
     <xacro:property name="wheel_yoff" value="${base_width/2 + wheel_width/2 + wheel_ygap}"/>
     <xacro:property name="wheel_zoff" value="0.05" />
+    <!-- 관성(Inertia) 계산 매크로 추가 (Gazebo 시뮬레이션용 필수) -->
+    <xacro:macro name="box_inertia" params="m w h d">
+        <inertial>
+            <origin xyz="0 0 0" rpy="${pi/2} 0 ${pi/2}"/>
+            <mass value="${m}"/>
+            <inertia ixx="${(m/12) * (h*h + d*d)}" ixy="0.0" ixz="0.0" iyy="${(m/12) * (w*w + d*d)}" iyz="0.0" izz="${(m/12) * (w*w + h*h)}"/>
+        </inertial>
+    </xacro:macro>
+    <xacro:macro name="cylinder_inertia" params="m r h">
+        <inertial>
+            <origin xyz="0 0 0" rpy="${pi/2} 0 0"/>
+            <mass value="${m}"/>
+            <inertia ixx="${(m/12) * (3*r*r + h*h)}" ixy="0" ixz="0" iyy="${(m/12) * (3*r*r + h*h)}" iyz="0" izz="${(m/2) * (r*r)}"/>
+        </inertial>
+    </xacro:macro>
     <!-- 2. 재질(Material) 정의 -->
     <material name="blue">
@@ -31,4 +46,10 @@
             <material name="blue"/>
         </visual>
+        <collision>
+            <geometry>
+                <box size="${base_length} ${base_width} ${base_height}"/>
+            </geometry>
+        </collision>
+        <xacro:box_inertia m="15.0" w="${base_width}" d="${base_length}" h="${base_height}"/>
     </link>
     <!-- 4. 바퀴 매크로 (Wheel Macro) -->
@@ -44,4 +65,11 @@
                  <material name="black"/>
             </visual>
+            <collision>
+                <origin xyz="0 0 0" rpy="${pi/2} 0 0"/>
+                <geometry>
+                    <cylinder radius="${wheel_radius}" length="${wheel_width}"/>
+                </geometry>
+            </collision>
+            <xacro:cylinder_inertia m="1.0" r="${wheel_radius}" h="${base_height}"/>
         </link>
         <!-- 회전 확인용 인디케이터 (별도 링크로 분리) -->
@@ -57,4 +85,5 @@
                 <material name="white"/>
             </visual>
+            <xacro:box_inertia m="0.01" w="0.01" d="0.03" h="${wheel_width + 0.002}"/>
         </link>
         <joint name="${prefix}_indicator_joint" type="fixed">
@@ -77,3 +106,29 @@
     <xacro:wheel prefix="rear_left" x_reflect="-1" y_reflect="1" />
     <xacro:wheel prefix="rear_right" x_reflect="-1" y_reflect="-1" />
+    <!-- 6. Gazebo 구동 플러그인 (Skid Steer Drive) -->
+    <!-- 이 플러그인이 cmd_vel 토픽을 구독하여 4개의 바퀴 관절을 회전시킵니다. -->
+    <gazebo>
+        <plugin name="skid_steer_drive" filename="libgazebo_ros_diff_drive.so">
+            <!-- 바퀴 개수 설정 -->
+            <num_wheel_pairs>2</num_wheel_pairs>
+            <!-- 왼쪽/오른쪽 조인트 매핑 -->
+            <left_joint>front_left_joint</left_joint>
+            <left_joint>rear_left_joint</left_joint>
+            <right_joint>front_right_joint</right_joint>
+            <right_joint>rear_right_joint</right_joint>
+            <!-- 로봇의 물리적 치수 (동역학 계산에 사용됨) -->
+            <!-- wheel_separation: 좌우 바퀴 중심 간의 거리 -->
+            <wheel_separation>${base_width + wheel_width + 2*wheel_ygap}</wheel_separation>
+            <wheel_diameter>${2 * wheel_radius}</wheel_diameter>
+            <!-- 제어 파라미터 -->
+            <max_wheel_torque>20</max_wheel_torque>
+            <max_wheel_acceleration>1.0</max_wheel_acceleration>
+            <!-- ROS 2 인터페이스 설정 -->
+            <publish_odom>true</publish_odom>
+            <publish_odom_tf>true</publish_odom_tf>
+            <publish_wheel_tf>true</publish_wheel_tf>
+            <odometry_frame>odom</odometry_frame>
+            <robot_base_frame>base_link</robot_base_frame>
+        </plugin>
+    </gazebo>
 </robot>
